File: RW_board/motor_driver.kicad_sch (KiCad schematic)
At the start: 22 parts, among them IC1 MCT8316Z0RQRGFRQ1

Commit message: Revert "Completed motor driver schematic"
This reverts commit 6eff020a4600c20233f645a88c0bbf96158f60b4.
Parts:
- removed C6: 150u, Capacitor_SMD:CP_Elec_6.3x7.7, symbol Device:C_Polarized
- removed C8: 100n, Capacitor_SMD:C_0402_1005Metric, symbol Device:C
- removed D1, D2, D3: LED, symbol Device:LED
- removed R10, R8: 330, symbol Device:R
- removed R7: 5.1k, symbol Device:R
- removed R9: 10k, symbol Device:R
- R1, R4: value 5.1k -> 10k
Connections:
- net GNDPWR is gone; now on net GND: C3.2, C4.2, IC1.12 (PGND_1), IC1.15 (PGND_2), IC1.18 (PGND_3)
- net FB_BK: no longer names the net of C7.1, IC1.3 (FB_BK), R3.1
- net Motor_24V renamed Motor_12V
- net SW_BK: no longer names the net of IC1.5 (SW_BK), R3.2
Other:
- moved on the sheet: C5, R5, R6
