File: RW_board/buck_boost.kicad_sch (KiCad schematic)
At the start: 45 parts, among them IC201 MAX44284WAUT+T, Q201 BSZ300N15NS5ATMA1, U201 LM5022MM

Commit message: Bom completed and generated, minor PCB adjustments
Parts:
- C219: renamed from C1; Voltage rating (none) -> 35V
- L201: DKPN (none) -> 2457-XGL4040-223MEC-ND
- Q201: Mouser Part Number (none) -> 726-BSZ300N15NS5ATMA
- R1: Mouser Part Number (none) -> 710-560112110083
- R201: Mouser Part Number (none) -> 710-560112110032
- R202: Mouser Part Number (none) -> 710-560112110020
- R203: Mouser Part Number (none) -> 652-CRT0402FZ3011GLF
- R204: Mouser Part Number (none) -> 710-560112110185
- R205: Mouser Part Number (none) -> 603-RT0402BRD076K9L
- R206: Mouser Part Number (none) -> 710-560112110022
- R207: Manufacturer_Part_Number (none) -> RL1220S-R39-F; Mouser Part Number (none) -> 754-RL1220S-R39-F
- R208, R210: Mouser Part Number (none) -> 710-560112110178
- R209: Mouser Part Number (none) -> 652-CRT0402FZ1331GLF
- R211: Mouser Part Number (none) -> 710-560112110116
- R212, R214: Mouser Part Number (none) -> 710-560112110012
- R213: footprint Capacitor_SMD:C_0603_1608Metric -> Resistor_SMD:R_0603_1608Metric; Mouser Part Number (none) -> 603-PE0603DRF570R02L
- U201: Mouser Part Number (none) -> 926-LM5022MMX/NOPB
Changed lines of the file:
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@@
 			)
 		)
+		(property "Mouser Part Number" "710-560112110012 "
+			(at 275.59 63.5 0)
+			(effects
+				(font
+					(size 1.27 1.27)
+				)
+				(hide yes)
+			)
+		)
 		(pin "1"
 		)
@@
 			)
 		)
+		(property "Mouser Part Number" "710-560112110178 "
+			(at 232.41 29.21 0)
+			(effects
+				(font
+					(size 1.27 1.27)
+				)
+				(hide yes)
+			)
+		)
 		(pin "1"
 		)
@@
 		(on_board yes)
 		(dnp no)
-		(property "Reference" "C1"
-			(at 264.922 116.84 0)
+		(property "Reference" "C219"
+			(at 266.954 117.094 0)
 			(effects
 				(font
@@
 			)
 		)
+		(property "Voltage rating" "35V"
+			(at 266.7 114.3 0)
+			(effects
+				(font
+					(size 1.27 1.27)
+				)
+				(hide yes)
+			)
+		)
 		(pin "1"
 		)
@@
 			(project "RW_board"
 				(path "/ff273890-9ca6-499d-9c73-a93557b69e48/818fd1d9-2c7b-4967-b4fa-637005b787d9"
-					(reference "C1")
+					(reference "C219")
 					(unit 1)
 				)
@@
 			)
 		)
+		(property "Mouser Part Number" "652-CRT0402FZ3011GLF "
+			(at 68.58 85.09 0)
+			(effects
+				(font
+					(size 1.27 1.27)
+				)
+				(hide yes)
+			)
+		)
 		(pin "1"
 		)
@@
 			)
 		)
+		(property "DKPN" "2457-XGL4040-223MEC-ND "
+			(at 93.98 50.8 0)
+			(effects
+				(font
+					(size 1.27 1.27)
+				)
+				(hide yes)
+			)
+		)
 		(pin "2"
 		)
@@
 			)
 		)
+		(property "Mouser Part Number" "710-560112110083 "
+			(at 226.06 49.53 0)
+			(effects
+				(font
+					(size 1.27 1.27)
+				)
+				(hide yes)
+			)
+		)
 		(pin "1"
 		)
@@
 			)
 		)
-		(property "Footprint" "Capacitor_SMD:C_0603_1608Metric"
+		(property "Footprint" "Resistor_SMD:R_0603_1608Metric"
 			(at 267.97 41.402 90)
 			(effects
@@
 			)
 		)
+		(property "Mouser Part Number" "603-PE0603DRF570R02L "
+			(at 267.97 43.18 0)
+			(effects
+				(font
+					(size 1.27 1.27)
+				)
+				(hide yes)
+			)
+		)
 		(pin "1"
 		)
@@
 			)
 		)
-		(property "Mouser Part Number" ""
+		(property "Mouser Part Number" "726-BSZ300N15NS5ATMA "
 			(at 191.77 538.1 0)
 			(effects
@@
 			)
 		)
+		(property "Mouser Part Number" "926-LM5022MMX/NOPB "
+			(at 91.44 74.93 0)
+			(effects
+				(font
+					(size 1.27 1.27)
+				)
+				(hide yes)
+			)
+		)
 		(pin "2"
 		)
@@
 			)
 		)
+		(property "Mouser Part Number" "603-RT0402BRD076K9L "
+			(at 118.11 58.42 0)
+			(effects
+				(font
+					(size 1.27 1.27)
+				)
+				(hide yes)
+			)
+		)
 		(pin "1"
 		)
@@
 			)
 		)
+		(property "Mouser Part Number" "710-560112110012 "
+			(at 261.62 63.5 0)
+			(effects
+				(font
+					(size 1.27 1.27)
+				)
+				(hide yes)
+			)
+		)
 		(pin "1"
 		)
@@
 			)
 		)
+		(property "Mouser Part Number" "710-560112110022 "
+			(at 135.89 58.42 0)
+			(effects
+				(font
+					(size 1.27 1.27)
+				)
+				(hide yes)
+			)
+		)
 		(pin "1"
 		)
@@
 			)
 		)
+		(property "Mouser Part Number" "652-CRT0402FZ1331GLF "
+			(at 226.06 87.63 0)
+			(effects
+				(font
+					(size 1.27 1.27)
+				)
+				(hide yes)
+			)
+		)
 		(pin "1"
 		)
@@
 			)
 		)
+		(property "Mouser Part Number" "710-560112110178 "
+			(at 226.06 68.58 0)
+			(effects
+				(font
+					(size 1.27 1.27)
+				)
+				(hide yes)
+			)
+		)
 		(pin "1"
 		)
@@
 			)
 		)
+		(property "Mouser Part Number" "710-560112110020 "
+			(at 68.58 59.69 0)
+			(effects
+				(font
+					(size 1.27 1.27)
+				)
+				(hide yes)
+			)
+		)
 		(pin "1"
 		)
@@
 			)
 		)
+		(property "Manufacturer_Part_Number" "RL1220S-R39-F "
+			(at 146.05 66.04 0)
+			(effects
+				(font
+					(size 1.27 1.27)
+				)
+				(hide yes)
+			)
+		)
+		(property "Mouser Part Number" "754-RL1220S-R39-F "
+			(at 146.05 66.04 0)
+			(effects
+				(font
+					(size 1.27 1.27)
+				)
+				(hide yes)
+			)
+		)
 		(pin "1"
 		)
@@
 			)
 		)
+		(property "Mouser Part Number" "710-560112110116 "
+			(at 252.73 29.21 0)
+			(effects
+				(font
+					(size 1.27 1.27)
+				)
+				(hide yes)
+			)
+		)
 		(pin "1"
 		)
@@
 			)
 		)
+		(property "Mouser Part Number" "710-560112110185 "
+			(at 113.03 91.44 0)
+			(effects
+				(font
+					(size 1.27 1.27)
+				)
+				(hide yes)
+			)
+		)
 		(pin "1"
 		)
@@
 			(at 59.69 85.09 0)
 			(effects
+				(font
+					(size 1.27 1.27)
+				)
+				(hide yes)
+			)
+		)
+		(property "Mouser Part Number" "710-560112110032"
+			(at 59.69 85.09 0)
+			(effects
