File: RW_board/mcu.kicad_sch (KiCad schematic)
At the start: 25 parts, among them J1 USB4105-GF-A, J2 20021521-00010T4LF, SW1 SW_Push, U1 ATSAMD21G18A-M, Y1 32.768KHz

Commit message: Initial board layout
Parts:
- removed Y1: 32.768KHz, 830105946101, symbol RW_Imports:830105946101
- added Y401: 830105946101, 830105946101, symbol RW_Imports:830105946101
- D402: renamed from D5; footprint (none) -> LED_SMD:LED_0603_1608Metric
- J401: renamed from J1; footprint USB4105-GF-A:GCT_USB4105-GF-A -> RW_Imports:GCT_USB4105-GF-A
- R406: renamed from R16; footprint (none) -> Resistor_SMD:R_0402_1005Metric
- SW401: renamed from SW1; footprint (none) -> Button_Switch_SMD:SW_SPST_FSMSM; DKPN (none) -> CKN10384TR-ND
- renumbered C12 to C401, C11 to C402, C9 to C403, C10 to C404, C13 to C405, C14 to C406, C15 to C407, C16 to C408, C17 to C409, C18 to C410, D4 to D401, J2 to J402, R18 to R401, R14 to R402, R13 to R403, R11 to R404, R17 to R405, R12 to R407, R15 to R408, U1 to U401
Connections:
- net at C403.2, U401.1 (PA00): now also Y401.1
- net at C404.2, U401.2 (PA01): now also Y401.2 (CRYSTAL_2)
- net ADC3: now reaches U401.9 (PA04)

Commit message: Added logo, TVS diode, made test production files
Parts:
- added D403: PRTR5V0U2X,215, PRTR5V0U2X, symbol RW_Imports:PRTR5V0U2X,215
Connections:
- net +3.3V: now also D403.4 (supply_voltage)
- net GND: now also D403.1 (ground)
- net UART_RX: now also D403.2 (input/output_1)
- net UART_TX: now also D403.3 (input/output_2)

Commit message: via fix
Connections:
- net GND: now also D401.1 (ground)
- net SHIELD: no longer D401.1 (ground)
Changed lines of the file:
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@@
+	(wire
+		(pts
+			(xy 97.79 130.81) (xy 97.79 134.62)
+		)
+		(stroke
+			(width 0)
+			(type default)
+		)
+	)
 	(wire
 		(pts
@@
 	(label "MCU_nRESET"
 		(at 254 123.19 180)
-		(effects
-			(font
-				(size 1.27 1.27)
-			)
-			(justify right bottom)
-		)
-	)
-	(label "SHIELD"
-		(at 97.79 130.81 180)
 		(effects
 			(font
@@
 					(unit 1)
 				)
+			)
+		)
+	)
+	(symbol
+		(lib_id "power:GND")
+		(at 97.79 134.62 0)
+		(unit 1)
+		(exclude_from_sim no)
+		(in_bom yes)
+		(on_board yes)
+		(dnp no)
+		(fields_autoplaced yes)
+		(property "Reference" "#PWR0417"
+			(at 97.79 140.97 0)
+			(effects
+				(font
+					(size 1.27 1.27)
+				)
+				(hide yes)
+			)
+		)
+		(property "Value" "GND"
+			(at 97.79 139.7 0)
+			(effects
+				(font
+					(size 1.27 1.27)
+				)
+			)
+		)
+		(property "Footprint" ""
+			(at 97.79 134.62 0)
+			(effects
+				(font
+					(size 1.27 1.27)
+				)
+				(hide yes)
+			)
+		)
+		(property "Datasheet" ""
+			(at 97.79 134.62 0)
+			(effects
+				(font
+					(size 1.27 1.27)
+				)
+				(hide yes)
+			)
+		)
+		(property "Description" "Power symbol creates a global label with name \"GND\" , ground"
+			(at 97.79 134.62 0)
+			(effects
+				(font
+					(size 1.27 1.27)
+				)
+				(hide yes)
+			)
+		)
+		(pin "1"
+		)
+		(instances
+			(project "RW_board"
+				(path "/ff273890-9ca6-499d-9c73-a93557b69e48/d46f2397-fda0-49de-8aef-b2135a54a0d5"
+					(reference "#PWR0417")
+					(unit 1)
+				)

Commit message: Add part numbers
Parts:
- C401, C402: Voltage Rating 30V -> (none); Voltage rating (none) -> 35V
- C405: Mouser Part Number (none) -> 81-GRM155R6YA105KE1J; Voltage rating 30V -> 35V
- C406, C407, C408, C409, C410: Voltage rating 30V -> 35V
Changed lines of the file:
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@@
 	(label "SHIELD"
 		(at 93.98 114.3 180)
-		(fields_autoplaced yes)
 		(effects
 			(font
@@
 	(label "MCU_nRESET"
 		(at 41.91 45.72 0)
-		(fields_autoplaced yes)
 		(effects
 			(font
@@
 	(label "SWDIO"
 		(at 135.89 121.92 0)
-		(fields_autoplaced yes)
 		(effects
 			(font
@@
 	(label "VBUS"
 		(at 91.44 78.74 180)
-		(fields_autoplaced yes)
 		(effects
 			(font
@@
 	(label "MCU_nRESET"
 		(at 254 123.19 180)
-		(fields_autoplaced yes)
 		(effects
 			(font
@@
 	(label "VBUS"
 		(at 97.79 128.27 180)
-		(fields_autoplaced yes)
 		(effects
 			(font
@@
 	(label "SWCLK"
 		(at 254 115.57 180)
-		(fields_autoplaced yes)
 		(effects
 			(font
@@
 	(label "D_N"
 		(at 40.64 88.9 0)
-		(fields_autoplaced yes)
 		(effects
 			(font
@@
 	(label "SWCLK"
 		(at 135.89 119.38 0)
-		(fields_autoplaced yes)
 		(effects
 			(font
@@
 	(label "D_P"
 		(at 41.91 128.27 0)
-		(fields_autoplaced yes)
 		(effects
 			(font
@@
 	(label "D_N"
 		(at 91.44 88.9 180)
-		(fields_autoplaced yes)
 		(effects
 			(font
@@
 	(label "SWDIO"
 		(at 238.76 113.03 180)
-		(fields_autoplaced yes)
 		(effects
 			(font
@@
 	(label "MCU_nRESET"
 		(at 132.08 127 0)
-		(fields_autoplaced yes)
 		(effects
 			(font
@@
 	(label "D_N"
 		(at 41.91 130.81 0)
-		(fields_autoplaced yes)
 		(effects
 			(font
@@
 	(label "D_N"
 		(at 139.7 104.14 0)
-		(fields_autoplaced yes)
 		(effects
 			(font
@@
 	(label "D_P"
 		(at 139.7 106.68 0)
-		(fields_autoplaced yes)
 		(effects
 			(font
@@
 	(label "D_P"
 		(at 91.44 86.36 180)
-		(fields_autoplaced yes)
 		(effects
 			(font
@@
 	(label "D_P"
 		(at 40.64 86.36 0)
-		(fields_autoplaced yes)
 		(effects
 			(font
@@
 		(shape input)
 		(at 184.15 68.58 0)
-		(fields_autoplaced yes)
 		(effects
 			(font
@@
 		(shape input)
 		(at 138.43 99.06 180)
-		(fields_autoplaced yes)
 		(effects
 			(font
@@
 		(shape input)
 		(at 138.43 83.82 180)
-		(fields_autoplaced yes)
 		(effects
 			(font
@@
 		(shape input)
 		(at 184.15 71.12 0)
-		(fields_autoplaced yes)
 		(effects
 			(font
@@
 		(shape input)
 		(at 186.69 101.6 0)
-		(fields_autoplaced yes)
 		(effects
 			(font
@@
 		(shape input)
 		(at 184.15 50.8 0)
-		(fields_autoplaced yes)
 		(effects
 			(font
@@
 		(shape input)
 		(at 184.15 48.26 0)
-		(fields_autoplaced yes)
 		(effects
 			(font
@@
 		(shape input)
 		(at 138.43 101.6 180)
-		(fields_autoplaced yes)
 		(effects
 			(font
@@
 		(shape input)
 		(at 138.43 96.52 180)
-		(fields_autoplaced yes)
 		(effects
 			(font
@@
 		(shape input)
 		(at 142.24 71.12 180)
-		(fields_autoplaced yes)
 		(effects
 			(font
@@
 		(shape input)
 		(at 215.9 30.48 180)
-		(fields_autoplaced yes)
 		(effects
 			(font
@@
 		(shape output)
 		(at 142.24 48.26 180)
-		(fields_autoplaced yes)
 		(effects
 			(font
@@
 		(shape input)
 		(at 143.51 53.34 180)
-		(fields_autoplaced yes)
 		(effects
 			(font
@@
 		(shape input)
 		(at 138.43 86.36 180)
-		(fields_autoplaced yes)
 		(effects
 			(font
@@
 		(shape input)
 		(at 138.43 93.98 180)
-		(fields_autoplaced yes)
 		(effects
 			(font
@@
 		(shape input)
 		(at 44.45 173.99 180)
-		(fields_autoplaced yes)
 		(effects
 			(font
@@
 		(shape input)
 		(at 142.24 68.58 180)
-		(fields_autoplaced yes)
 		(effects
 			(font
@@
 		(shape input)
 		(at 44.45 171.45 180)
-		(fields_autoplaced yes)
 		(effects
 			(font
@@
 		(shape input)
 		(at 138.43 91.44 180)
-		(fields_autoplaced yes)
 		(effects
 			(font
@@
 		(shape input)
 		(at 186.69 99.06 0)
-		(fields_autoplaced yes)
 		(effects
 			(font
@@
 			)
 		)
-		(property "Voltage rating" "30V"
+		(property "Voltage rating" "35V"
 			(at 199.39 41.91 0)
 			(effects
@@
 			)
 		)
-		(property "Voltage rating" "30V"
+		(property "Voltage rating" "35V"
+			(at 151.13 29.21 0)
+			(effects
+				(font
+					(size 1.27 1.27)
+				)
+				(hide yes)
+			)
+		)
+		(property "Mouser Part Number" "81-GRM155R6YA105KE1J "
 			(at 151.13 29.21 0)
 			(effects
@@
 			)
 		)
-		(property "Voltage rating" "30V"
+		(property "Voltage rating" "35V"
 			(at 234.95 41.91 0)
 			(effects
@@
 			)
 		)
-		(property "Voltage rating" "30V"
+		(property "Voltage rating" "35V"
 			(at 210.82 41.91 0)
 			(effects
@@
 			)
 		)
-		(property "Voltage Rating" "30V"
+		(property "Voltage Rating" ""
 			(at 57.15 52.07 90)
+			(effects
+				(font
+					(size 1.27 1.27)
+				)
+				(hide yes)
+			)
+		)
+		(property "Voltage rating" "35V"
+			(at 57.15 52.07 0)
 			(effects
 				(font
@@
 			)
 		)
-		(property "Voltage rating" "30V"
+		(property "Voltage rating" "35V"
 			(at 223.52 41.91 0)
 			(effects
@@
 			)
 		)
-		(property "Voltage Rating" "30V"
+		(property "Voltage Rating" ""
 			(at 95.25 106.68 90)
+			(effects
+				(font
+					(size 1.27 1.27)
+				)
+				(hide yes)
+			)
+		)
+		(property "Voltage rating" "35V"
+			(at 95.25 106.68 0)
 			(effects
 				(font
@@
 			)
 		)
-		(property "Voltage rating" "30V"
+		(property "Voltage rating" "35V"
 			(at 246.38 41.91 0)
 			(effects
