File: RW_board/mcu.kicad_sch (KiCad schematic)
At the start: 26 parts, among them J401 USB4105-GF-A, J402 20021521-00010T4LF, SW401 SW_Push, U401 ATSAMD21G18A-M, Y401 830105946101

Commit message: Bom completed and generated, minor PCB adjustments
Parts:
- C401, C407, C408, C409, C410: Mouser Part Number (none) -> 81-GRM155R61H104KE9J
- C402: Mouser Part Number (none) -> 81-GRM155R71H472JA1D
- C403, C404: Mouser Part Number (none) -> 81-GRM1555C1H200JA1D
- C406: Mouser Part Number (none) -> 81-GRM155R61A475MEAD
- D402: Mouser Part Number (none) -> 720-P412Q2T136A8J802
- J401: Mouser Part Number (none) -> 640-USB4105-GF-A
- J402: Mouser Part Number (none) -> 649-221521-00010T4LF
- R401, R405: Mouser Part Number (none) -> 652-CR0402FX-5101GLF
- R402: Mouser Part Number (none) -> 710-560112110020
- R403: Mouser Part Number (none) -> 710-560112110231
- R404: Mouser Part Number (none) -> 710-560112110033
- R406: value 330 -> 330R; Mouser Part Number (none) -> 710-560112110231
- R407: Mouser Part Number (none) -> 710-560112110014
- R408: Mouser Part Number (none) -> 710-560112110012
- SW401: Mouser Part Number (none) -> 611-RS-282G05A3-SMRT
- U401: Mouser Part Number (none) -> 556-ATSAMD21G18A-MUT
Changed lines of the file:
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@@
 			)
 		)
+		(property "Mouser Part Number" "81-GRM155R61A475MEAD "
+			(at 199.39 41.91 0)
+			(effects
+				(font
+					(size 1.27 1.27)
+				)
+				(hide yes)
+			)
+		)
 		(pin "1"
 		)
@@
 			)
 		)
-		(property "Mouser Part Number" ""
+		(property "Mouser Part Number" "649-221521-00010T4LF "
 			(at 226.06 607.95 0)
 			(effects
@@
 			)
 		)
+		(property "Mouser Part Number" "652-CR0402FX-5101GLF "
+			(at 95.25 83.82 0)
+			(effects
+				(font
+					(size 1.27 1.27)
+				)
+				(hide yes)
+			)
+		)
 		(pin "2"
 		)
@@
 			)
 		)
+		(property "Mouser Part Number" "81-GRM155R61H104KE9J "
+			(at 234.95 41.91 0)
+			(effects
+				(font
+					(size 1.27 1.27)
+				)
+				(hide yes)
+			)
+		)
 		(pin "1"
 		)
@@
 			)
 		)
+		(property "Mouser Part Number" "710-560112110014 "
+			(at 234.95 123.19 0)
+			(effects
+				(font
+					(size 1.27 1.27)
+				)
+				(hide yes)
+			)
+		)
 		(pin "2"
 		)
@@
 			)
 		)
+		(property "Mouser Part Number" "710-560112110020 "
+			(at 57.15 36.83 0)
+			(effects
+				(font
+					(size 1.27 1.27)
+				)
+				(hide yes)
+			)
+		)
 		(pin "2"
 		)
@@
 			)
 		)
+		(property "Mouser Part Number" "710-560112110012 "
+			(at 243.84 107.95 0)
+			(effects
+				(font
+					(size 1.27 1.27)
+				)
+				(hide yes)
+			)
+		)
 		(pin "2"
 		)
@@
 			)
 		)
+		(property "Mouser Part Number" "710-560112110033 "
+			(at 93.98 101.6 0)
+			(effects
+				(font
+					(size 1.27 1.27)
+				)
+				(hide yes)
+			)
+		)
 		(pin "2"
 		)
@@
 			)
 		)
+		(property "Mouser Part Number" "81-GRM155R61H104KE9J "
+			(at 210.82 41.91 0)
+			(effects
+				(font
+					(size 1.27 1.27)
+				)
+				(hide yes)
+			)
+		)
 		(pin "1"
 		)
@@
 			)
 		)
+		(property "Mouser Part Number" "81-GRM155R61H104KE9J "
+			(at 57.15 52.07 0)
+			(effects
+				(font
+					(size 1.27 1.27)
+				)
+				(hide yes)
+			)
+		)
 		(pin "2"
 		)
@@
 			)
 		)
+		(property "Mouser Part Number" "652-CR0402FX-5101GLF "
+			(at 39.37 97.79 0)
+			(effects
+				(font
+					(size 1.27 1.27)
+				)
+				(hide yes)
+			)
+		)
 		(pin "2"
 		)
@@
 			)
 		)
+		(property "Mouser Part Number" "81-GRM155R61H104KE9J "
+			(at 223.52 41.91 0)
+			(effects
+				(font
+					(size 1.27 1.27)
+				)
+				(hide yes)
+			)
+		)
 		(pin "1"
 		)
@@
 			)
 		)
+		(property "Mouser Part Number" "81-GRM155R71H472JA1D "
+			(at 95.25 106.68 0)
+			(effects
+				(font
+					(size 1.27 1.27)
+				)
+				(hide yes)
+			)
+		)
 		(pin "2"
 		)
@@
 			)
 		)
+		(property "Mouser Part Number" "720-P412Q2T136A8J802 "
+			(at 203.2 80.01 0)
+			(effects
+				(font
+					(size 1.27 1.27)
+				)
+				(hide yes)
+			)
+		)
 		(pin "1"
 		)
@@
 			)
 		)
+		(property "Mouser Part Number" "556-ATSAMD21G18A-MUT "
+			(at 163.83 83.82 0)
+			(effects
+				(font
+					(size 1.27 1.27)
+				)
+				(hide yes)
+			)
+		)
 		(pin "37"
 		)
@@
 			)
 		)
+		(property "Mouser Part Number" "710-560112110231 "
+			(at 77.47 50.8 0)
+			(effects
+				(font
+					(size 1.27 1.27)
+				)
+				(hide yes)
+			)
+		)
 		(pin "2"
 		)
@@
 			)
 		)
+		(property "Mouser Part Number" "81-GRM155R61H104KE9J "
+			(at 246.38 41.91 0)
+			(effects
+				(font
+					(size 1.27 1.27)
+				)
+				(hide yes)
+			)
+		)
 		(pin "1"
 		)
@@
 			)
 		)
-		(property "Value" "330"
+		(property "Value" "330R"
 			(at 204.978 72.136 0)
 			(effects
@@
 			)
 		)
+		(property "Mouser Part Number" "710-560112110231 "
+			(at 203.2 71.12 0)
+			(effects
+				(font
+					(size 1.27 1.27)
+				)
+				(hide yes)
+			)
+		)
 		(pin "2"
 		)
@@
 			)
 		)
+		(property "Mouser Part Number" "81-GRM1555C1H200JA1D "
+			(at 116.84 45.72 0)
+			(effects
+				(font
+					(size 1.27 1.27)
+				)
+				(hide yes)
+			)
+		)
 		(pin "1"
 		)
@@
 			)
 		)
+		(property "Mouser Part Number" "611-RS-282G05A3-SMRT "
+			(at 66.04 45.72 0)
+			(effects
+				(font
+					(size 1.27 1.27)
+				)
+				(hide yes)
+			)
+		)
 		(pin "1"
 		)
@@
 			)
 		)
+		(property "Mouser Part Number" "640-USB4105-GF-A "
+			(at 66.04 88.9 0)
+			(effects
+				(font
+					(size 1.27 1.27)
+				)
+				(hide yes)
+			)
+		)
 		(pin "A7"
 		)
@@
 			(at 116.84 34.29 0)
 			(effects
+				(font
+					(size 1.27 1.27)
+				)
+				(hide yes)
+			)
+		)
+		(property "Mouser Part Number" "81-GRM1555C1H200JA1D "
+			(at 116.84 34.29 0)
+			(effects
